File: KiCad_L/KiCad_L.kicad_sch (KiCad schematic)
At the start: 0 parts

Commit message: feat: Leftの回路データが完成
Parts:
- added C1, C2: C, Capacitor_SMD:C_0805_2012Metric, symbol Device:C
- added D1, D10, D11, D12, D13, D14, D15, D16, D17, D18, D19, D2, D20, D21, D22, D23, D24, D25, D26, D27, D28, D29, D3, D31, D4, D5, D6, D7, D8, D9: 1N4148W, Diode_SMD:D_SOD-123, symbol Diode:1N4148W
- added D30, D32: LED, LED_SMD:LED_0805_2012Metric, symbol Device:LED
- added J1: AudioJack3_SwitchTR, Connector_Audio:Jack_3.5mm_CUI_SJ1-3515N_Horizontal, symbol Connector_Audio:AudioJack3_SwitchTR
- added R1, R2: R, Resistor_SMD:R_0805_2012Metric, symbol Device:R
- added SW1: Esc, PCM_Switch_Keyboard_Hotswap_Kailh:SW_Hotswap_Kailh_Choc_V2_1.00u, symbol Switch:SW_Push
- added SW10: E, PCM_Switch_Keyboard_Hotswap_Kailh:SW_Hotswap_Kailh_Choc_V2_1.00u, symbol Switch:SW_Push
- added SW11: R, PCM_Switch_Keyboard_Hotswap_Kailh:SW_Hotswap_Kailh_Choc_V2_1.00u, symbol Switch:SW_Push
- added SW12: T, PCM_Switch_Keyboard_Hotswap_Kailh:SW_Hotswap_Kailh_Choc_V2_1.00u, symbol Switch:SW_Push
- added SW13: Ctrl, PCM_Switch_Keyboard_Hotswap_Kailh:SW_Hotswap_Kailh_Choc_V2_1.00u, symbol Switch:SW_Push
- added SW14: A, PCM_Switch_Keyboard_Hotswap_Kailh:SW_Hotswap_Kailh_Choc_V2_1.00u, symbol Switch:SW_Push
- added SW15: S, PCM_Switch_Keyboard_Hotswap_Kailh:SW_Hotswap_Kailh_Choc_V2_1.00u, symbol Switch:SW_Push
- added SW16: D, PCM_Switch_Keyboard_Hotswap_Kailh:SW_Hotswap_Kailh_Choc_V2_1.00u, symbol Switch:SW_Push
- added SW17: F, PCM_Switch_Keyboard_Hotswap_Kailh:SW_Hotswap_Kailh_Choc_V2_1.00u, symbol Switch:SW_Push
- added SW18: G, PCM_Switch_Keyboard_Hotswap_Kailh:SW_Hotswap_Kailh_Choc_V2_1.00u, symbol Switch:SW_Push
- added SW19: Shift, PCM_Switch_Keyboard_Hotswap_Kailh:SW_Hotswap_Kailh_Choc_V2_1.00u, symbol Switch:SW_Push
- added SW2: 1, PCM_Switch_Keyboard_Hotswap_Kailh:SW_Hotswap_Kailh_Choc_V2_1.00u, symbol Switch:SW_Push
- added SW20: Z, PCM_Switch_Keyboard_Hotswap_Kailh:SW_Hotswap_Kailh_Choc_V2_1.00u, symbol Switch:SW_Push
- added SW21: X, PCM_Switch_Keyboard_Hotswap_Kailh:SW_Hotswap_Kailh_Choc_V2_1.00u, symbol Switch:SW_Push
- added SW22: C, PCM_Switch_Keyboard_Hotswap_Kailh:SW_Hotswap_Kailh_Choc_V2_1.00u, symbol Switch:SW_Push
- added SW23: V, PCM_Switch_Keyboard_Hotswap_Kailh:SW_Hotswap_Kailh_Choc_V2_1.00u, symbol Switch:SW_Push
- added SW24: 6, PCM_Switch_Keyboard_Hotswap_Kailh:SW_Hotswap_Kailh_Choc_V2_1.00u, symbol Switch:SW_Push
- added SW25: Fn, PCM_Switch_Keyboard_Hotswap_Kailh:SW_Hotswap_Kailh_Choc_V2_1.00u, symbol Switch:SW_Push
- added SW26: Alt, PCM_Switch_Keyboard_Hotswap_Kailh:SW_Hotswap_Kailh_Choc_V2_1.00u, symbol Switch:SW_Push
- added SW27: Win, PCM_Switch_Keyboard_Hotswap_Kailh:SW_Hotswap_Kailh_Choc_V2_1.00u, symbol Switch:SW_Push
- added SW28: NoConv, PCM_Switch_Keyboard_Hotswap_Kailh:SW_Hotswap_Kailh_Choc_V2_1.00u, symbol Switch:SW_Push
- added SW29: Space, PCM_Switch_Keyboard_Hotswap_Kailh:SW_Hotswap_Kailh_Choc_V2_1.00u, symbol Switch:SW_Push
- added SW3: 2, PCM_Switch_Keyboard_Hotswap_Kailh:SW_Hotswap_Kailh_Choc_V2_1.00u, symbol Switch:SW_Push
- added SW4: 3, PCM_Switch_Keyboard_Hotswap_Kailh:SW_Hotswap_Kailh_Choc_V2_1.00u, symbol Switch:SW_Push
- added SW5: 4, PCM_Switch_Keyboard_Hotswap_Kailh:SW_Hotswap_Kailh_Choc_V2_1.00u, symbol Switch:SW_Push
- added SW6: 5, PCM_Switch_Keyboard_Hotswap_Kailh:SW_Hotswap_Kailh_Choc_V2_1.00u, symbol Switch:SW_Push
- added SW7: Tab, PCM_Switch_Keyboard_Hotswap_Kailh:SW_Hotswap_Kailh_Choc_V2_1.00u, symbol Switch:SW_Push
- added SW8: Q, PCM_Switch_Keyboard_Hotswap_Kailh:SW_Hotswap_Kailh_Choc_V2_1.00u, symbol Switch:SW_Push
- added SW9: W, PCM_Switch_Keyboard_Hotswap_Kailh:SW_Hotswap_Kailh_Choc_V2_1.00u, symbol Switch:SW_Push
- added U1: Sparkfun_Pro_Micro, Arduino:Sparkfun_Pro_Micro, symbol Arduino_g200kg:Sparkfun_Pro_Micro
Connections:
- new net: D4.2 (A), SW4.2
- new net: D16.2 (A), SW16.2
- new net: D32.2 (A), R2.1
- new net: R2.2, U1.13 (~D10/A10)
- new net: D14.2 (A), SW14.2
- new net: D18.2 (A), SW18.2
- new net: D9.2 (A), SW9.2
- new net: D17.2 (A), SW17.2
- new net: D23.2 (A), SW23.2
- new net: D11.2 (A), SW11.2
- new net: D28.2 (A), SW28.2
- new net: D24.2 (A), SW24.2
- new net: D8.2 (A), SW8.2
- new net: D6.2 (A), SW6.2
- new net: D3.2 (A), SW3.2
- new net: D19.2 (A), SW19.2
- new net: D7.2 (A), SW7.2
- new net: D25.2 (A), SW25.2
- new net: D26.2 (A), SW26.2
- new net: D12.2 (A), SW12.2
- new net: D2.2 (A), SW2.2
- new net: R1.1, U1.14 (D16)
- new net: D30.2 (A), R1.2
- new net: D21.2 (A), SW21.2
- new net: D29.2 (A), SW29.2
- new net: D22.2 (A), SW22.2
- new net: D10.2 (A), SW10.2
- new net: D1.2 (A), SW1.2
- new net: D20.2 (A), SW20.2
- new net: D5.2 (A), SW5.2
- new net: D27.2 (A), SW27.2
- new net: D15.2 (A), SW15.2
- new net: D13.2 (A), SW13.2
- new net +5V: C1.1, C2.1, D31.1 (K), J1.R, U1.12 (~D9/A9), U1.21 (VCC)
- new net Col0: SW1.1, SW13.1, SW19.1, SW25.1, SW7.1, U1.20 (D21/A3)
- new net Col1: SW14.1, SW2.1, SW20.1, SW26.1, SW8.1, U1.19 (D20/A2)
- new net Col2: SW15.1, SW21.1, SW27.1, SW3.1, SW9.1, U1.18 (D19/A1)
- new net Col3: SW10.1, SW16.1, SW22.1, SW28.1, SW4.1, U1.17 (D18/A0)
- new net Col4: SW11.1, SW17.1, SW23.1, SW29.1, SW5.1, U1.16 (D15)
- new net Col5: SW12.1, SW18.1, SW24.1, SW6.1, U1.15 (D14)
- new net GND: C1.2, C2.2, D30.1 (K), D31.2 (A), D32.1 (K), J1.S, U1.23 (GND), U1.3 (GND), U1.4 (GND)
- new net Row0: D1.1 (K), D2.1 (K), D3.1 (K), D4.1 (K), D5.1 (K), D6.1 (K), U1.7 (D4/A6)
- new net Row1: D10.1 (K), D11.1 (K), D12.1 (K), D7.1 (K), D8.1 (K), D9.1 (K), U1.8 (~D5)
- new net Row2: D13.1 (K), D14.1 (K), D15.1 (K), D16.1 (K), D17.1 (K), D18.1 (K), U1.9 (~D6/A7)
- new net Row3: D19.1 (K), D20.1 (K), D21.1 (K), D22.1 (K), D23.1 (K), D24.1 (K), U1.10 (D7)
- new net Row4: D25.1 (K), D26.1 (K), D27.1 (K), D28.1 (K), D29.1 (K), U1.11 (D8/A8)
- new net SCL: J1.T, U1.6 (~D3)
- new net SDA: U1.5 (D2)
- no-connect marks 0 -> 2
Other:
- note added: "分割判定フラグ （R側ではGNDに接続）"
- company: (none) -> 1x telescope
- title: (none) -> Just the Two of JIS - Left
