File: KiCad_Kailh_L_top/KiCad_Kailh_L_top.kicad_sch (KiCad schematic)
At the start: 67 parts, among them J1 AudioJack3_SwitchTR, SW1 Esc, SW10 E, SW11 R, SW12 T, SW13 Ctrl, SW14 A, SW15 S, SW16 D, SW17 F, SW18 G, SW19 Shift, SW2 1, SW20 Z, SW21 X, SW22 C, SW23 V, SW24 6, SW25 Fn, SW26 Alt, SW27 Win, SW28 NoConv, SW29 Space, SW3 2, SW4 3, SW5 4, SW6 5, SW7 Tab, SW8 Q, SW9 W, U1 Sparkfun_Pro_Micro

Commit message: feat: Leftの各データが完成
Parts:
- removed D30, D32: LED, LED_SMD:LED_0805_2012Metric, symbol Device:LED
- removed R2: R, Resistor_SMD:R_0805_2012Metric, symbol Device:R
- added D31: LED, LED_THT:LED_D5.0mm, symbol Device:LED
- D1, D10, D11, D12, D13, D14, D15, D16, D17, D18, D19, D2, D20, D21, D22, D23, D24, D25, D26, D27, D28, D29, D3, D4, D5, D6, D7, D8, D9: footprint Diode_SMD:D_SOD-123 -> Diode_SMD:D_SOD-323
- SW1, SW10, SW11, SW12, SW13, SW14, SW15, SW16, SW17, SW18, SW19, SW2, SW20, SW21, SW22, SW23, SW24, SW25, SW26, SW27, SW28, SW29, SW3, SW4, SW5, SW6, SW7, SW8, SW9: footprint PCM_Switch_Keyboard_Hotswap_Kailh:SW_Hotswap_Kailh_Choc_V2_1.00u -> KBD_BrownSugar:Switch_Hole
- renumbered D31 to D30
Connections:
- net +5V: now also R1.1
- net GND: now also D31.1 (K)
- net at U1.14 (D16): no longer R1.1
- net at R1.2: now also D31.2 (A)
- no-connect marks 2 -> 7
