File: KiCad_Cherry_L_pcb/KiCad_Cherry_L_pcb.kicad_sch (KiCad schematic)
At the start: 63 parts, among them J1 AudioJack3_SwitchTR, SW1 Esc, SW10 E, SW11 R, SW12 T, SW13 Ctrl, SW14 A, SW15 S, SW16 D, SW17 F, SW18 G, SW19 Shift, SW2 1, SW20 Z, SW21 X, SW22 C, SW23 V, SW24 6, SW25 Fn, SW26 Alt, SW27 Win, SW28 NoConv, SW29 Space, SW3 2, SW4 3, SW5 4, SW6 5, SW7 Tab, SW8 Q, SW9 W, U1 Sparkfun_Pro_Micro

Commit message: refactor: 作り直し
Parts:
- D30: footprint Diode_SMD:D_SOD-123 -> Diode_SMD:D_SOD-323
- SW1, SW10, SW11, SW12, SW14, SW15, SW16, SW17, SW18, SW2, SW20, SW21, SW22, SW23, SW24, SW3, SW4, SW5, SW6, SW8, SW9: footprint PCM_Switch_Keyboard_Kailh:SW_Kailh_Choc_V1_1.00u -> KBD_BrownSugar:CherryMX_Hotswap_via_1U
- SW13: footprint PCM_Switch_Keyboard_Kailh:SW_Kailh_Choc_V1_1.75u -> KBD_BrownSugar:CherryMX_Hotswap_via_1.75U
- SW19: footprint PCM_Switch_Keyboard_Kailh:SW_Kailh_Choc_V1_2.25u -> KBD_BrownSugar:CherryMX_Hotswap_via_2.25U
- SW25, SW26, SW27, SW28: footprint PCM_Switch_Keyboard_Kailh:SW_Kailh_Choc_V1_1.25u -> KBD_BrownSugar:CherryMX_Hotswap_via_1.25U
- SW29: footprint PCM_Switch_Keyboard_Kailh:SW_Kailh_Choc_V1_2.00u -> KBD_BrownSugar:CherryMX_Hotswap_via_2U
- SW7: footprint PCM_Switch_Keyboard_Kailh:SW_Kailh_Choc_V1_1.50u -> KBD_BrownSugar:CherryMX_Hotswap_via_1.5U
