File: KiCad_Kailh_L_pcb/KiCad_Kailh_L_pcb.kicad_sch (KiCad schematic)
At the start: 63 parts, among them J1 AudioJack3_SwitchTR, SW1 Esc, SW10 E, SW11 R, SW12 T, SW13 Ctrl, SW14 A, SW15 S, SW16 D, SW17 F, SW18 G, SW19 Shift, SW2 1, SW20 Z, SW21 X, SW22 C, SW23 V, SW24 6, SW25 Fn, SW26 Alt, SW27 Win, SW28 NoConv, SW29 Space, SW3 2, SW4 3, SW5 4, SW6 5, SW7 Tab, SW8 Q, SW9 W, U1 Sparkfun_Pro_Micro

Commit message: refactor: 作り直し
Parts:
- SW1, SW10, SW11, SW12, SW14, SW15, SW16, SW17, SW18, SW2, SW20, SW21, SW22, SW23, SW24, SW3, SW4, SW5, SW6, SW8, SW9: footprint PCM_Switch_Keyboard_Kailh:SW_Kailh_Choc_V1_1.00u -> PCM_Switch_Keyboard_Hotswap_Kailh:SW_Hotswap_Kailh_Choc_V2_1.00u
- SW13: footprint PCM_Switch_Keyboard_Kailh:SW_Kailh_Choc_V1_1.75u -> PCM_Switch_Keyboard_Hotswap_Kailh:SW_Hotswap_Kailh_Choc_V2_1.75u
- SW19: footprint PCM_Switch_Keyboard_Kailh:SW_Kailh_Choc_V1_2.25u -> PCM_Switch_Keyboard_Hotswap_Kailh:SW_Hotswap_Kailh_Choc_V2_2.25u
- SW25, SW26, SW27, SW28: footprint PCM_Switch_Keyboard_Kailh:SW_Kailh_Choc_V1_1.25u -> PCM_Switch_Keyboard_Hotswap_Kailh:SW_Hotswap_Kailh_Choc_V2_1.25u
- SW29: footprint PCM_Switch_Keyboard_Kailh:SW_Kailh_Choc_V1_2.00u -> PCM_Switch_Keyboard_Hotswap_Kailh:SW_Hotswap_Kailh_Choc_V2_2.00u
- SW7: footprint PCM_Switch_Keyboard_Kailh:SW_Kailh_Choc_V1_1.50u -> PCM_Switch_Keyboard_Hotswap_Kailh:SW_Hotswap_Kailh_Choc_V2_1.50u
Changed lines of the file:
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@@
 			)
 		)
-		(property "Footprint" "PCM_Switch_Keyboard_Kailh:SW_Kailh_Choc_V1_1.00u"
+		(property "Footprint" "PCM_Switch_Keyboard_Hotswap_Kailh:SW_Hotswap_Kailh_Choc_V2_1.00u"
 			(at 171.45 77.47 0)
 			(effects
@@
 			)
 		)
-		(property "Footprint" "PCM_Switch_Keyboard_Kailh:SW_Kailh_Choc_V1_1.00u"
+		(property "Footprint" "PCM_Switch_Keyboard_Hotswap_Kailh:SW_Hotswap_Kailh_Choc_V2_1.00u"
 			(at 95.25 77.47 0)
 			(effects
@@
 			)
 		)
-		(property "Footprint" "PCM_Switch_Keyboard_Kailh:SW_Kailh_Choc_V1_1.00u"
+		(property "Footprint" "PCM_Switch_Keyboard_Hotswap_Kailh:SW_Hotswap_Kailh_Choc_V2_1.00u"
 			(at 247.65 77.47 0)
 			(effects
@@
 			)
 		)
-		(property "Footprint" "PCM_Switch_Keyboard_Kailh:SW_Kailh_Choc_V1_1.00u"
+		(property "Footprint" "PCM_Switch_Keyboard_Hotswap_Kailh:SW_Hotswap_Kailh_Choc_V2_1.00u"
 			(at 133.35 52.07 0)
 			(effects
@@
 			)
 		)
-		(property "Footprint" "PCM_Switch_Keyboard_Kailh:SW_Kailh_Choc_V1_1.00u"
+		(property "Footprint" "PCM_Switch_Keyboard_Hotswap_Kailh:SW_Hotswap_Kailh_Choc_V2_1.00u"
 			(at 209.55 102.87 0)
 			(effects
@@
 			)
 		)
-		(property "Footprint" "PCM_Switch_Keyboard_Kailh:SW_Kailh_Choc_V1_1.00u"
+		(property "Footprint" "PCM_Switch_Keyboard_Hotswap_Kailh:SW_Hotswap_Kailh_Choc_V2_1.00u"
 			(at 209.55 52.07 0)
 			(effects
@@
 			)
 		)
-		(property "Footprint" "PCM_Switch_Keyboard_Kailh:SW_Kailh_Choc_V1_1.00u"
+		(property "Footprint" "PCM_Switch_Keyboard_Hotswap_Kailh:SW_Hotswap_Kailh_Choc_V2_1.00u"
 			(at 247.65 102.87 0)
 			(effects
@@
 			)
 		)
-		(property "Footprint" "PCM_Switch_Keyboard_Kailh:SW_Kailh_Choc_V1_1.00u"
+		(property "Footprint" "PCM_Switch_Keyboard_Hotswap_Kailh:SW_Hotswap_Kailh_Choc_V2_1.00u"
 			(at 133.35 26.67 0)
 			(effects
@@
 			)
 		)
-		(property "Footprint" "PCM_Switch_Keyboard_Kailh:SW_Kailh_Choc_V1_2.25u"
+		(property "Footprint" "PCM_Switch_Keyboard_Hotswap_Kailh:SW_Hotswap_Kailh_Choc_V2_2.25u"
 			(at 57.15 102.87 0)
 			(effects
@@
 			)
 		)
-		(property "Footprint" "PCM_Switch_Keyboard_Kailh:SW_Kailh_Choc_V1_1.25u"
+		(property "Footprint" "PCM_Switch_Keyboard_Hotswap_Kailh:SW_Hotswap_Kailh_Choc_V2_1.25u"
 			(at 57.15 128.27 0)
 			(effects
@@
 			)
 		)
-		(property "Footprint" "PCM_Switch_Keyboard_Kailh:SW_Kailh_Choc_V1_1.00u"
+		(property "Footprint" "PCM_Switch_Keyboard_Hotswap_Kailh:SW_Hotswap_Kailh_Choc_V2_1.00u"
 			(at 95.25 26.67 0)
 			(effects
@@
 			)
 		)
-		(property "Footprint" "PCM_Switch_Keyboard_Kailh:SW_Kailh_Choc_V1_1.50u"
+		(property "Footprint" "PCM_Switch_Keyboard_Hotswap_Kailh:SW_Hotswap_Kailh_Choc_V2_1.50u"
 			(at 57.15 52.07 0)
 			(effects
@@
 			)
 		)
-		(property "Footprint" "PCM_Switch_Keyboard_Kailh:SW_Kailh_Choc_V1_1.00u"
+		(property "Footprint" "PCM_Switch_Keyboard_Hotswap_Kailh:SW_Hotswap_Kailh_Choc_V2_1.00u"
 			(at 171.45 26.67 0)
 			(effects
@@
 			)
 		)
-		(property "Footprint" "PCM_Switch_Keyboard_Kailh:SW_Kailh_Choc_V1_1.25u"
+		(property "Footprint" "PCM_Switch_Keyboard_Hotswap_Kailh:SW_Hotswap_Kailh_Choc_V2_1.25u"
 			(at 95.25 128.27 0)
 			(effects
@@
 			)
 		)
-		(property "Footprint" "PCM_Switch_Keyboard_Kailh:SW_Kailh_Choc_V1_1.00u"
+		(property "Footprint" "PCM_Switch_Keyboard_Hotswap_Kailh:SW_Hotswap_Kailh_Choc_V2_1.00u"
 			(at 133.35 102.87 0)
 			(effects
@@
 			)
 		)
-		(property "Footprint" "PCM_Switch_Keyboard_Kailh:SW_Kailh_Choc_V1_1.25u"
+		(property "Footprint" "PCM_Switch_Keyboard_Hotswap_Kailh:SW_Hotswap_Kailh_Choc_V2_1.25u"
 			(at 171.45 128.27 0)
 			(effects
@@
 			)
 		)
-		(property "Footprint" "PCM_Switch_Keyboard_Kailh:SW_Kailh_Choc_V1_2.00u"
+		(property "Footprint" "PCM_Switch_Keyboard_Hotswap_Kailh:SW_Hotswap_Kailh_Choc_V2_2.00u"
 			(at 209.55 128.27 0)
 			(effects
@@
 			)
 		)
-		(property "Footprint" "PCM_Switch_Keyboard_Kailh:SW_Kailh_Choc_V1_1.00u"
+		(property "Footprint" "PCM_Switch_Keyboard_Hotswap_Kailh:SW_Hotswap_Kailh_Choc_V2_1.00u"
 			(at 57.15 26.67 0)
 			(effects
@@
 			)
 		)
-		(property "Footprint" "PCM_Switch_Keyboard_Kailh:SW_Kailh_Choc_V1_1.00u"
+		(property "Footprint" "PCM_Switch_Keyboard_Hotswap_Kailh:SW_Hotswap_Kailh_Choc_V2_1.00u"
 			(at 247.65 52.07 0)
 			(effects
@@
 			)
 		)
-		(property "Footprint" "PCM_Switch_Keyboard_Kailh:SW_Kailh_Choc_V1_1.00u"
+		(property "Footprint" "PCM_Switch_Keyboard_Hotswap_Kailh:SW_Hotswap_Kailh_Choc_V2_1.00u"
 			(at 209.55 26.67 0)
 			(effects
@@
 			)
 		)
-		(property "Footprint" "PCM_Switch_Keyboard_Kailh:SW_Kailh_Choc_V1_1.00u"
+		(property "Footprint" "PCM_Switch_Keyboard_Hotswap_Kailh:SW_Hotswap_Kailh_Choc_V2_1.00u"
 			(at 133.35 77.47 0)
 			(effects
@@
 			)
 		)
-		(property "Footprint" "PCM_Switch_Keyboard_Kailh:SW_Kailh_Choc_V1_1.00u"
+		(property "Footprint" "PCM_Switch_Keyboard_Hotswap_Kailh:SW_Hotswap_Kailh_Choc_V2_1.00u"
 			(at 171.45 52.07 0)
 			(effects
@@
 			)
 		)
-		(property "Footprint" "PCM_Switch_Keyboard_Kailh:SW_Kailh_Choc_V1_1.25u"
+		(property "Footprint" "PCM_Switch_Keyboard_Hotswap_Kailh:SW_Hotswap_Kailh_Choc_V2_1.25u"
 			(at 133.35 128.27 0)
 			(effects
@@
 			)
 		)
-		(property "Footprint" "PCM_Switch_Keyboard_Kailh:SW_Kailh_Choc_V1_1.00u"
+		(property "Footprint" "PCM_Switch_Keyboard_Hotswap_Kailh:SW_Hotswap_Kailh_Choc_V2_1.00u"
 			(at 247.65 26.67 0)
 			(effects
@@
 			)
 		)
-		(property "Footprint" "PCM_Switch_Keyboard_Kailh:SW_Kailh_Choc_V1_1.75u"
+		(property "Footprint" "PCM_Switch_Keyboard_Hotswap_Kailh:SW_Hotswap_Kailh_Choc_V2_1.75u"
 			(at 57.15 77.47 0)
 			(effects
@@
 			)
 		)
-		(property "Footprint" "PCM_Switch_Keyboard_Kailh:SW_Kailh_Choc_V1_1.00u"
+		(property "Footprint" "PCM_Switch_Keyboard_Hotswap_Kailh:SW_Hotswap_Kailh_Choc_V2_1.00u"
 			(at 209.55 77.47 0)
 			(effects
@@
 			)
 		)
-		(property "Footprint" "PCM_Switch_Keyboard_Kailh:SW_Kailh_Choc_V1_1.00u"
+		(property "Footprint" "PCM_Switch_Keyboard_Hotswap_Kailh:SW_Hotswap_Kailh_Choc_V2_1.00u"
 			(at 95.25 102.87 0)
 			(effects
@@
 			)
 		)
-		(property "Footprint" "PCM_Switch_Keyboard_Kailh:SW_Kailh_Choc_V1_1.00u"
+		(property "Footprint" "PCM_Switch_Keyboard_Hotswap_Kailh:SW_Hotswap_Kailh_Choc_V2_1.00u"
 			(at 171.45 102.87 0)
 			(effects
@@
 			)
 		)
-		(property "Footprint" "PCM_Switch_Keyboard_Kailh:SW_Kailh_Choc_V1_1.00u"
+		(property "Footprint" "PCM_Switch_Keyboard_Hotswap_Kailh:SW_Hotswap_Kailh_Choc_V2_1.00u"
 			(at 95.25 52.07 0)
 			(effects

Commit message: feat: Resetピンを追加
Parts:
- added J2: Reset, Connector_PinHeader_1.00mm:PinHeader_1x01_P1.00mm_Vertical, symbol Connector:Conn_01x01_Pin
Connections:
- net at U1.22 (RST): now also J2.1 (Pin_1)
Changed lines of the file:
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@@
+	)
+	(symbol
+		(lib_id "Connector:Conn_01x01_Pin")
+		(at 80.01 165.1 0)
+		(mirror y)
+		(unit 1)
+		(exclude_from_sim no)
+		(in_bom yes)
+		(on_board yes)
+		(dnp no)
+		(property "Reference" "J2"
+			(at 85.09 162.56 0)
+			(effects
+				(font
+					(size 1.27 1.27)
+				)
+			)
+		)
+		(property "Value" "Reset"
+			(at 85.09 165.1 0)
+			(effects
+				(font
+					(size 1.27 1.27)
+				)
+			)
+		)
+		(property "Footprint" "Connector_PinHeader_1.00mm:PinHeader_1x01_P1.00mm_Vertical"
+			(at 80.01 165.1 0)
+			(effects
+				(font
+					(size 1.27 1.27)
+				)
+				(hide yes)
+			)
+		)
+		(property "Datasheet" "~"
+			(at 80.01 165.1 0)
+			(effects
+				(font
+					(size 1.27 1.27)
+				)
+				(hide yes)
+			)
+		)
+		(property "Description" "Generic connector, single row, 01x01, script generated"
+			(at 80.01 165.1 0)
+			(effects
+				(font
+					(size 1.27 1.27)
+				)
+				(hide yes)
+			)
+		)
+		(pin "1"
+		)
+		(instances
+			(project "KiCad_Kailh_L_pcb"
+				(path "/63624602-85c8-4a35-8071-08b2ca90618c"
+					(reference "J2")
+					(unit 1)
+				)
+			)
+		)
 	)
 	(symbol

Commit message: feat: Rightのガワを用意
Parts:
- added D31: LED, LED_SMD:LED_0805_2012Metric, symbol Device:LED
- added R1: 10k, Resistor_SMD:R_0805_2012Metric, symbol Device:R
Connections:
- net GND: now also R1.1
- net at U1.2 (D0/RX): now also D31.2 (A)
- new net: D31.1 (K), R1.2
- no-connect marks 7 -> 6
