File: KiCad_Cherry_L_others/top/KiCad_Cherry_L_top.kicad_pcb (KiCad board)
At the start: 2 copper layers, 138.1 x 100 mm, 43 parts, among them SW1 Esc, SW10 E, SW11 R, SW12 T, SW13 Ctrl, SW14 A, SW15 S, SW16 D, SW17 F, SW18 G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

Commit message: feat: Rightのガワを用意
Parts:
- removed SW19: Shift, KBD_BrownSugar:Switch_Hole
- removed SW29: Space, KBD_BrownSugar:Switch_Hole
- added REF**: Stabilizer 2U, KBD_BrownSugar:Stabilizer_MX_Plate_Mount_2U, F.Cu at (197.6, 133.3)
- added REF**: Stabilizer 2U, KBD_BrownSugar:Stabilizer_MX_Plate_Mount_2U, F.Cu at (104.8, 114.3)
