File: KiCad_Cherry_L_others/bottom/KiCad_Cherry_L_pcb.kicad_pcb (KiCad board)
At the start: 2 copper layers, 138.1 x 100 mm, 0 parts

Commit message: feat: ガワがすべて完成
Other:
- outline, holes or cut-outs redrawn
Changed lines of the file:
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@@
 	)
 	(net 0 "")
-	(gr_arc
-		(start 80.96253 50.00625)
-		(mid 82.357436 46.638677)
+	(gr_line
+		(start 80.9625 50.00625)
+		(end 80.9625 140.49375)
+		(stroke
+			(width 0.05)
+			(type default)
+		)
+		(layer "Edge.Cuts")
+	)
+	(gr_arc
+		(start 80.9625 50.00625)
+		(mid 82.357404 46.638654)
 		(end 85.725 45.24375)
 		(stroke
@@
 			(type default)
 		)
-		(locked yes)
-		(layer "Edge.Cuts")
-	)
-	(gr_line
-		(start 80.962568 54.173483)
-		(end 80.962501 50.00625)
-		(stroke
-			(width 0.05)
-			(type default)
-		)
-		(locked yes)
-		(layer "Edge.Cuts")
-	)
-	(gr_line
-		(start 80.962568 54.173483)
-		(end 80.9625 140.49372)
-		(stroke
-			(width 0.05)
-			(type default)
-		)
-		(locked yes)
-		(layer "Edge.Cuts")
-	)
-	(gr_circle
-		(center 83.34382 66.675056)
-		(end 83.939133 66.079743)
-		(stroke
-			(width 0.05)
-			(type default)
-		)
-		(fill no)
-		(locked yes)
+		(layer "Edge.Cuts")
+	)
+	(gr_circle
+		(center 83.34382 50.006292)
+		(end 83.939133 50.006292)
+		(stroke
+			(width 0.05)
+			(type default)
+		)
+		(fill no)
+		(layer "Edge.Cuts")
+	)
+	(gr_circle
+		(center 83.34382 69.056308)
+		(end 83.939133 69.056308)
+		(stroke
+			(width 0.05)
+			(type default)
+		)
+		(fill no)
 		(layer "Edge.Cuts")
 	)
 	(gr_circle
 		(center 83.34382 95.25008)
-		(end 83.939133 94.654767)
-		(stroke
-			(width 0.05)
-			(type default)
-		)
-		(fill no)
-		(locked yes)
+		(end 83.939133 95.25008)
+		(stroke
+			(width 0.05)
+			(type default)
+		)
+		(fill no)
 		(layer "Edge.Cuts")
 	)
 	(gr_circle
 		(center 83.34382 123.825104)
-		(end 83.939133 123.229791)
-		(stroke
-			(width 0.05)
-			(type default)
-		)
-		(fill no)
-		(locked yes)
+		(end 83.939133 123.825104)
+		(stroke
+			(width 0.05)
+			(type default)
+		)
+		(fill no)
 		(layer "Edge.Cuts")
 	)
 	(gr_arc
 		(start 85.725 145.25625)
-		(mid 82.357482 143.861303)
-		(end 80.96269 140.49372)
-		(stroke
-			(width 0.05)
-			(type default)
-		)
-		(locked yes)
+		(mid 82.357404 143.861346)
+		(end 80.9625 140.49375)
+		(stroke
+			(width 0.05)
+			(type default)
+		)
 		(layer "Edge.Cuts")
 	)
 	(gr_circle
 		(center 92.868828 47.62504)
-		(end 93.464141 47.029727)
-		(stroke
-			(width 0.05)
-			(type default)
-		)
-		(fill no)
-		(locked yes)
+		(end 93.464141 47.62504)
+		(stroke
+			(width 0.05)
+			(type default)
+		)
+		(fill no)
 		(layer "Edge.Cuts")
 	)
 	(gr_circle
 		(center 92.868828 142.87512)
-		(end 93.464141 142.279807)
-		(stroke
-			(width 0.05)
-			(type default)
-		)
-		(fill no)
-		(locked yes)
+		(end 93.464141 142.87512)
+		(stroke
+			(width 0.05)
+			(type default)
+		)
+		(fill no)
 		(layer "Edge.Cuts")
 	)
 	(gr_circle
 		(center 130.96886 47.62504)
-		(end 131.564173 47.029727)
-		(stroke
-			(width 0.05)
-			(type default)
-		)
-		(fill no)
-		(locked yes)
+		(end 131.564173 47.62504)
+		(stroke
+			(width 0.05)
+			(type default)
+		)
+		(fill no)
 		(layer "Edge.Cuts")
 	)
 	(gr_circle
 		(center 130.96886 142.87512)
-		(end 131.564173 142.279807)
-		(stroke
-			(width 0.05)
-			(type default)
-		)
-		(fill no)
-		(locked yes)
+		(end 131.564173 142.87512)
+		(stroke
+			(width 0.05)
+			(type default)
+		)
+		(fill no)
 		(layer "Edge.Cuts")
 	)
 	(gr_circle
 		(center 169.068892 47.62504)
-		(end 169.664205 47.029727)
-		(stroke
-			(width 0.05)
-			(type default)
-		)
-		(fill no)
-		(locked yes)
+		(end 169.664205 47.62504)
+		(stroke
+			(width 0.05)
+			(type default)
+		)
+		(fill no)
 		(layer "Edge.Cuts")
 	)
 	(gr_circle
 		(center 169.068892 142.87512)
-		(end 169.664205 142.279807)
-		(stroke
-			(width 0.05)
-			(type default)
-		)
-		(fill no)
-		(locked yes)
+		(end 169.664205 142.87512)
+		(stroke
+			(width 0.05)
+			(type default)
+		)
+		(fill no)
 		(layer "Edge.Cuts")
 	)
 	(gr_circle
 		(center 207.168924 47.62504)
-		(end 207.764237 47.029727)
-		(stroke
-			(width 0.05)
-			(type default)
-		)
-		(fill no)
-		(locked yes)
+		(end 207.764237 47.62504)
+		(stroke
+			(width 0.05)
+			(type default)
+		)
+		(fill no)
 		(layer "Edge.Cuts")
 	)
 	(gr_circle
 		(center 207.168924 142.87512)
-		(end 207.764237 142.279807)
-		(stroke
-			(width 0.05)
-			(type default)
-		)
-		(fill no)
-		(locked yes)
+		(end 207.764237 142.87512)
+		(stroke
+			(width 0.05)
+			(type default)
+		)
+		(fill no)
 		(layer "Edge.Cuts")
 	)
@@
 			(type default)
 		)
-		(locked yes)
 		(layer "Edge.Cuts")
 	)
 	(gr_arc
 		(start 214.3125 45.24375)
-		(mid 217.687952 46.64633)
-		(end 219.075172 50.028124)
-		(stroke
-			(width 0.05)
-			(type default)
-		)
-		(locked yes)
+		(mid 217.680096 46.638654)
+		(end 219.075 50.00625)
+		(stroke
+			(width 0.05)
+			(type default)
+		)
 		(layer "Edge.Cuts")
 	)
@@
 			(type default)
 		)
-		(locked yes)
 		(layer "Edge.Cuts")
 	)
 	(gr_circle
 		(center 216.693932 66.675056)
-		(end 217.289245 66.079743)
-		(stroke
-			(width 0.05)
-			(type default)
-		)
-		(fill no)
-		(locked yes)
-		(layer "Edge.Cuts")
-	)
-	(gr_circle
-		(center 216.693932 95.25008)
-		(end 217.289245 94.654767)
-		(stroke
-			(width 0.05)
-			(type default)
-		)
-		(fill no)
-		(locked yes)
-		(layer "Edge.Cuts")
-	)
-	(gr_circle
-		(center 216.693932 123.825104)
-		(end 217.289245 123.229791)
-		(stroke
-			(width 0.05)
-			(type default)
-		)
-		(fill no)
-		(locked yes)
-		(layer "Edge.Cuts")
-	)
-	(gr_line
-		(start 219.075 50.028123)
-		(end 219.075184 118.467287)
-		(stroke
-			(width 0.05)
-			(type default)
-		)
-		(locked yes)
+		(end 217.289245 66.675056)
+		(stroke
+			(width 0.05)
+			(type default)
+		)
+		(fill no)
+		(layer "Edge.Cuts")
+	)
+	(gr_circle
+		(center 216.693932 105.965714)
+		(end 217.289245 105.965714)
+		(stroke
+			(width 0.05)
+			(type default)
+		)
+		(fill no)
+		(layer "Edge.Cuts")
+	)
+	(gr_circle
+		(center 216.693932 122.634478)
+		(end 217.289245 122.634478)
+		(stroke
+			(width 0.05)
+			(type default)
+		)
+		(fill no)
 		(layer "Edge.Cuts")
 	)
 	(gr_arc
 		(start 219.075 140.49375)
-		(mid 217.680127 143.861359)
-		(end 214.3125 145.256188)
-		(stroke
-			(width 0.05)
-			(type default)
-		)
-		(locked yes)
-		(layer "Edge.Cuts")
-	)
-	(gr_line
-		(start 219.075184 118.467287)
-		(end 219.075 140.49375)
-		(stroke
-			(width 0.05)
-			(type default)
-		)
-		(locked yes)
-		(layer "Edge.Cuts")
-	)
+		(mid 217.680096 143.861346)
+		(end 214.3125 145.25625)
+		(stroke
+			(width 0.05)
+			(type default)
+		)
+		(layer "Edge.Cuts")
+	)
+	(gr_line
+		(start 219.075 140.49375)
+		(end 219.075 50.00625)
+		(stroke
+			(width 0.05)
+			(type default)
+		)
+		(layer "Edge.Cuts")
+	)
