File: KiCad_Cherry_R_others/top/KiCad_Cherry_R_top.kicad_pcb (KiCad board)
At the start: 2 copper layers, 188.7 x 100 mm, 56 parts, among them SW1 7, SW10 I, SW11 O, SW12 P, SW13 [, SW14 ], SW15 H, SW16 J, SW17 K, SW18 L, SW19 ;, SW2 8, SW20 ', SW21 \, SW22 B, SW23 N, SW24 M, SW25 ,, SW26 ., SW27 /, SW28 Shift, SW29 Space, SW3 9, SW30 Conv, SW31 Win, SW32 Fn, SW33 ←, SW34 ↑, SW35 ↓, SW36 BS, SW37 Enter, SW38 Home, SW39 End, SW4 0, SW40 →, SW41 Free, SW42 PrtSc, SW5 -, SW6 =, SW7 `, SW8 Y, SW9 U

Commit message: feat: ガワがすべて完成
Parts:
- removed the REF** at (35.7, 85.7)
- removed SW29: Space, KBD_BrownSugar:Switch_Hole
- added REF**: MountingHole_2.2mm_M2, MountingHole:MountingHole_2.2mm_M2, F.Cu at (35.1, 69.1)
- added REF**: Stabilizer 2U, KBD_BrownSugar:Stabilizer_MX_Plate_Mount_2U, F.Cu at (61.9, 124.0)
- added REF**: MountingHole_2.2mm_M2, MountingHole:MountingHole_2.2mm_M2, F.Cu at (219.1, 59.5)
- added REF**: MountingHole_2.2mm_M2, MountingHole:MountingHole_2.2mm_M2, F.Cu at (35.1, 85.7)
- moved REF** 9.53 mm to (219.1, 95.2)
- moved REF** 3.62 mm to (35.1, 41.7)
- moved REF** 2.45 mm to (35.1, 123.8)
- moved REF** 2.38 mm to (219.1, 123.8)
- moved REF** 1.19 mm to (219.1, 41.7)
- turned SW15 to 180 degrees
- turned SW16 to 180 degrees
- turned SW17 to 180 degrees
- turned SW18 to 180 degrees
- turned SW19 to 180 degrees
- turned SW20 to 180 degrees
- turned SW21 to 180 degrees
