File: KiCad_Kailh_L_others/top/KiCad_Kailh_L_top.kicad_pcb (KiCad board)
At the start: 2 copper layers, 138.1 x 100 mm, 43 parts, among them SW1 Esc, SW10 E, SW11 R, SW12 T, SW13 Ctrl, SW14 A, SW15 S, SW16 D, SW17 F, SW18 G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

Commit message: feat: ガワがすべて完成
Parts:
- removed the REF** at (197.6, 133.3)
- removed the REF** at (104.8, 114.3)
- added H2: MountingHole_2.2mm_M2, MountingHole:MountingHole_2.2mm_M2, F.Cu at (83.3, 50.0)
- added REF**: Stabilizer 2U, KBD_BrownSugar:Stabilizer_Choc_V1_Plate_Mount_2U, F.Cu at (197.6, 133.3)
- added REF**: Stabilizer 2U, KBD_BrownSugar:Stabilizer_Choc_V1_Plate_Mount_2U, F.Cu at (104.8, 114.3)
- added SW19: Shift, KBD_BrownSugar:Switch_Hole, F.Cu at (104.8, 114.3)
- added SW29: Space, KBD_BrownSugar:Switch_Hole, F.Cu at (197.6, 133.3)
- moved H2 10.7 mm to (216.7, 106.0)
- moved H7 2.38 mm to (83.3, 69.1)
- moved H14 1.19 mm to (216.7, 122.6)
- turned SW13 to 0 degrees
- turned SW14 to 0 degrees
- turned SW15 to 0 degrees
- turned SW16 to 0 degrees
- turned SW17 to 0 degrees
- turned SW18 to 0 degrees
- turned SW20 to 180 degrees
- turned SW21 to 180 degrees
- turned SW22 to 180 degrees
- turned SW23 to 180 degrees
Other:
- outline, holes or cut-outs redrawn
