File: KiCad_Kailh_R_others/top/KiCad_Kailh_R_top.kicad_pcb (KiCad board)
At the start: 2 copper layers, 188.7 x 100 mm, 56 parts, among them SW1 7, SW10 I, SW11 O, SW12 P, SW13 [, SW14 ], SW15 H, SW16 J, SW17 K, SW18 L, SW19 ;, SW2 8, SW20 ', SW21 \, SW22 B, SW23 N, SW24 M, SW25 ,, SW26 ., SW27 /, SW28 Shift, SW29 Space, SW3 9, SW30 Conv, SW31 Win, SW32 Fn, SW33 ←, SW34 ↑, SW35 ↓, SW36 BS, SW37 Enter, SW38 Home, SW39 End, SW4 0, SW40 →, SW41 Free, SW42 PrtSc, SW5 -, SW6 =, SW7 `, SW8 Y, SW9 U

Commit message: feat: ガワがすべて完成
Parts:
- removed the REF** at (35.7, 45.2)
- removed the REF** at (35.7, 85.7)
- removed the REF** at (219.1, 42.9)
- removed the REF** at (35.7, 126.2)
- added REF**: MountingHole_2.2mm_M2, MountingHole:MountingHole_2.2mm_M2, F.Cu at (35.1, 88.1)
- added REF**: MountingHole_2.2mm_M2, MountingHole:MountingHole_2.2mm_M2, F.Cu at (35.1, 72.6)
- added REF**: MountingHole_2.2mm_M2, MountingHole:MountingHole_2.2mm_M2, F.Cu at (35.1, 126.2)
- added REF**: MountingHole_2.2mm_M2, MountingHole:MountingHole_2.2mm_M2, F.Cu at (219.1, 40.5)
- added REF**: MountingHole_2.2mm_M2, MountingHole:MountingHole_2.2mm_M2, F.Cu at (219.1, 59.5)
- added REF**: Stabilizer 2U, KBD_BrownSugar:Stabilizer_Choc_V1_Plate_Mount_2U, F.Cu at (61.9, 124.0)
- added REF**: MountingHole_2.2mm_M2, MountingHole:MountingHole_2.2mm_M2, F.Cu at (35.1, 45.2)
- turned SW15 to 180 degrees
- turned SW16 to 180 degrees
- turned SW17 to 180 degrees
- turned SW18 to 180 degrees
- turned SW19 to 180 degrees
- turned SW20 to 180 degrees
- turned SW21 to 180 degrees
- turned SW38 to 180 degrees
- turned SW40 to 180 degrees
