File: KiCad_Kailh_R_pcb/KiCad_Kailh_R_pcb.kicad_pcb (KiCad board)
At the start: 2 copper layers, 188.7 x 100 mm, 106 parts, among them J1 AudioJack3_SwitchTR, J2 Reset, SW1 7, SW10 I, SW11 O, SW12 P, SW13 [, SW14 ], SW15 H, SW16 J, SW17 K, SW18 L, SW19 ;, SW2 8, SW20 ', SW21 \, SW22 B, SW23 N, SW24 M, SW25 ,, SW26 ., SW27 /, SW28 Shift, SW29 Space, SW3 9, SW30 Conv, SW31 Win, SW32 Fn, SW33 ←, SW34 ↑, SW35 ↓, SW36 BS, SW37 Enter, SW38 Home, SW39 End, SW4 0, SW40 →, SW41 Free, SW42 PrtSc, SW5 -, SW6 =, SW7 `, SW8 Y, SW9 U, U1 Sparkfun_Pro_Micro

Commit message: feat: ガワがすべて完成
Parts:
- added REF**: MountingHole_2.2mm_M2, MountingHole:MountingHole_2.2mm_M2, F.Cu at (35.1, 72.6)
- added REF**: MountingHole_2.2mm_M2, MountingHole:MountingHole_2.2mm_M2, F.Cu at (219.1, 59.5)
- moved J1 14.4 mm to (38.0, 80.2)
- moved R1 8.37 mm to (34.8, 66.1)
- moved D44 7.22 mm to (41.7, 67.9)
- moved REF** 2.45 mm to (35.1, 88.1)
- moved REF** 2.38 mm to (219.1, 40.5)
- moved U1 0.83 mm to (184.6, 42.3)
- moved REF** 0.60 mm to (35.1, 126.2)
- moved REF** 0.60 mm to (35.1, 45.2)
- turned SW15 to 180 degrees
- turned SW16 to 180 degrees
- turned SW17 to 180 degrees
- turned SW18 to 180 degrees
- turned SW19 to 180 degrees
- turned SW20 to 180 degrees
- turned SW21 to 180 degrees
